File: 3V3-step-down.kicad_sch (KiCad schematic)
At the start: 6 parts, among them U7 TPS62175DQC

Commit message: Polish
Parts:
- renumbered C28 to C30, C29 to C31, L2 to L3, R45 to R47, R46 to R48, U7 to U8
Changed lines of the file:
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@@
 		(on_board yes)
 		(dnp no)
-		(property "Reference" "L2"
+		(property "Reference" "L3"
 			(at 144.78 84.074 90)
 			(effects
@@
 		(on_board yes)
 		(dnp no)
-		(property "Reference" "R45"
+		(property "Reference" "R47"
 			(at 154.178 95.3516 0)
 			(effects
@@
 		(on_board yes)
 		(dnp no)
-		(property "Reference" "#PWR068"
+		(property "Reference" "#PWR071"
 			(at 128.27 118.11 0)
 			(effects
@@
 		(on_board yes)
 		(dnp no)
-		(property "Reference" "C28"
+		(property "Reference" "C30"
 			(at 107.95 95.25 0)
 			(effects
@@
 		(on_board yes)
 		(dnp no)
-		(property "Reference" "R46"
+		(property "Reference" "R48"
 			(at 154.178 105.5116 0)
 			(effects
@@
 		(on_board yes)
 		(dnp no)
-		(property "Reference" "#PWR069"
+		(property "Reference" "#PWR072"
 			(at 152.4 119.38 0)
 			(effects
@@
 		(on_board yes)
 		(dnp no)
-		(property "Reference" "U7"
+		(property "Reference" "U8"
 			(at 129.54 82.1182 0)
 			(effects
@@
 		(on_board yes)
 		(dnp no)
-		(property "Reference" "#FLG05"
+		(property "Reference" "#FLG06"
 			(at 152.4 85.725 0)
 			(effects
@@
 		(on_board yes)
 		(dnp no)
-		(property "Reference" "C29"
+		(property "Reference" "C31"
 			(at 168.021 95.3516 0)
 			(effects
@@
 		(on_board yes)
 		(dnp no)
-		(property "Reference" "#PWR067"
+		(property "Reference" "#PWR070"
 			(at 107.95 109.22 0)
 			(effects
