File: LED_lowSide_driver.kicad_sch (KiCad schematic)
At the start: 3 parts, among them Q17 IRLML0030

Commit message: Polish
Parts:
- renumbered Q17 to Q18, R41 to R43, R42 to R44
Changed lines of the file:
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@@
 		(on_board yes)
 		(dnp no)
-		(property "Reference" "#PWR065"
+		(property "Reference" "#PWR066"
 			(at 142.24 109.22 0)
 			(effects
@@
 		(on_board yes)
 		(dnp no)
-		(property "Reference" "R42"
+		(property "Reference" "R44"
 			(at 132.08 97.79 90)
 			(effects
@@
 		(on_board yes)
 		(dnp no)
-		(property "Reference" "Q17"
+		(property "Reference" "Q18"
 			(at 143.51 86.36 0)
 			(effects
@@
 		(on_board yes)
 		(dnp no)
-		(property "Reference" "R41"
+		(property "Reference" "R43"
 			(at 125.73 88.9 90)
 			(effects
