File: alarm-clock_v3.kicad_sch (KiCad schematic)
At the start: 100 parts, among them J1 Photoresistor, J2 Vibration, J3 ESP, J4 ButtonPCB, J5 SWD, J6 XT30, J7 LED strip, Q1 BC846C, Q2 FDN306P, Q3 FDS2734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

Commit message: Polish
Parts:
- added TP1: 35V, TestPoint:TestPoint_THTPad_D1.5mm_Drill0.7mm, symbol Connector:TestPoint
- added TP2: GND, TestPoint:TestPoint_THTPad_D1.5mm_Drill0.7mm, symbol Connector:TestPoint
Connections:
- net GND: now also TP2.1
- net at C20.1, D4.1 (K), D5.1 (A1)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: now also TP1.1
Other:
- moved on the sheet: C24, D16, D17, D18, D19, D20, D21, D22, D23, D24, J2, J3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
