File: high-side-switch.kicad_sch (KiCad schematic)
At the start: 5 parts, among them Q4 BC846, Q5 BC856

Commit message: Polish
Parts:
- renumbered Q4 to Q10, Q5 to Q11, R23 to R32, R24 to R33, R25 to R34
Changed lines of the file:
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@@
 		(dnp no)
 		(fields_autoplaced yes)
-		(property "Reference" "Q4"
+		(property "Reference" "Q10"
 			(at 138.43 105.4099 0)
 			(effects
@@
 		(on_board yes)
 		(dnp no)
-		(property "Reference" "R25"
+		(property "Reference" "R34"
 			(at 135.89 96.52 90)
 			(effects
@@
 		(on_board yes)
 		(dnp no)
-		(property "Reference" "R24"
+		(property "Reference" "R33"
 			(at 135.89 86.36 90)
 			(effects
@@
 		(on_board yes)
 		(dnp no)
-		(property "Reference" "R23"
+		(property "Reference" "R32"
 			(at 121.92 106.68 90)
 			(effects
@@
 		(on_board yes)
 		(dnp no)
-		(property "Reference" "Q5"
+		(property "Reference" "Q11"
 			(at 154.94 91.4401 0)
 			(effects
@@
 		(dnp no)
 		(fields_autoplaced yes)
-		(property "Reference" "#PWR058"
+		(property "Reference" "#PWR061"
 			(at 135.89 120.65 0)
 			(effects
