File: alarm-clock_v3.kicad_pcb (KiCad board)
At the start: 2 copper layers, 0 parts

Commit message: Add PCB
Parts:
- added BT1: 9V 6LR61, Connector_Molex:Molex_PicoBlade_53047-0210_1x02_P1.25mm_Vertical, B.Cu at (144.0, 134.7)
- added C1: 100n 35V, Capacitor_SMD:C_0603_1608Metric_Pad1.08x0.95mm_HandSolder, B.Cu at (139.6, 117.2)
- added C10: 1n, Capacitor_SMD:C_0603_1608Metric_Pad1.08x0.95mm_HandSolder, B.Cu at (143.9, 105.7)
- added C11: 220n 35V, Capacitor_SMD:C_0805_2012Metric_Pad1.18x1.45mm_HandSolder, B.Cu at (137.1, 105.7)
- added C12: 100n, Capacitor_SMD:C_0603_1608Metric_Pad1.08x0.95mm_HandSolder, B.Cu at (157.0, 115.0)
- added C13: 1u, Capacitor_SMD:C_0603_1608Metric_Pad1.08x0.95mm_HandSolder, B.Cu at (164.2, 118.8)
- added C14: 10n, Capacitor_SMD:C_0603_1608Metric_Pad1.08x0.95mm_HandSolder, B.Cu at (164.2, 117.2)
- added C15: 10u 16V, Capacitor_SMD:C_0805_2012Metric_Pad1.18x1.45mm_HandSolder, B.Cu at (133.6, 106.9)
- added C16: 1u, Capacitor_SMD:C_0603_1608Metric_Pad1.08x0.95mm_HandSolder, B.Cu at (158.4, 102.7)
- added C17: 100n, Capacitor_SMD:C_0603_1608Metric_Pad1.08x0.95mm_HandSolder, B.Cu at (158.4, 104.2)
- added C18: 10n, Capacitor_SMD:C_0805_2012Metric_Pad1.18x1.45mm_HandSolder, B.Cu at (138.1, 111.7)
- added C19: 100n, Capacitor_SMD:C_0603_1608Metric_Pad1.08x0.95mm_HandSolder, F.Cu at (152.6, 113.3)
- added C2: 47n, Capacitor_SMD:C_0603_1608Metric_Pad1.08x0.95mm_HandSolder, B.Cu at (142.3, 109.2)
- added C20: 1µ 50V, Capacitor_SMD:C_0805_2012Metric_Pad1.18x1.45mm_HandSolder, B.Cu at (129.4, 102.8)
- added C21: 100n, Capacitor_SMD:C_0603_1608Metric_Pad1.08x0.95mm_HandSolder, F.Cu at (173.0, 113.6)
- added C22: 100n, Capacitor_SMD:C_0603_1608Metric_Pad1.08x0.95mm_HandSolder, F.Cu at (166.2, 117.2)
- added C23: 4u7, Capacitor_SMD:C_0603_1608Metric_Pad1.08x0.95mm_HandSolder, B.Cu at (181.3, 90.9)
- added C24: 100n, Capacitor_SMD:C_0603_1608Metric_Pad1.08x0.95mm_HandSolder, F.Cu at (165.0, 138.2)
- added C25: 100n 35V, Capacitor_SMD:C_0603_1608Metric_Pad1.08x0.95mm_HandSolder, B.Cu at (143.4, 130.5)
- added C26: 100n 35V, Capacitor_SMD:C_0603_1608Metric_Pad1.08x0.95mm_HandSolder, B.Cu at (141.8, 130.5)
- added C27: 22u 35V, Capacitor_SMD:C_0805_2012Metric_Pad1.18x1.45mm_HandSolder, B.Cu at (143.2, 123.9)
- added C28: 2u2 35V, Capacitor_SMD:C_0603_1608Metric_Pad1.08x0.95mm_HandSolder, F.Cu at (149.8, 129.5)
- added C29: 22u, Capacitor_SMD:C_0805_2012Metric_Pad1.18x1.45mm_HandSolder, F.Cu at (152.0, 126.8)
- added C3: 100n 35V, Capacitor_SMD:C_0603_1608Metric_Pad1.08x0.95mm_HandSolder, B.Cu at (139.6, 118.8)
- added C30: 2u2 35V, Capacitor_SMD:C_0603_1608Metric_Pad1.08x0.95mm_HandSolder, F.Cu at (159.8, 129.5)
- added C31: 22u, Capacitor_SMD:C_0805_2012Metric_Pad1.18x1.45mm_HandSolder, F.Cu at (162.0, 126.8)
- added C32: 100n, Capacitor_SMD:C_0603_1608Metric_Pad1.08x0.95mm_HandSolder, F.Cu at (175.8, 132.5)
- added C4: 10u, Capacitor_SMD:C_0805_2012Metric_Pad1.18x1.45mm_HandSolder, B.Cu at (156.0, 116.8)
- added C5: 22p, Capacitor_SMD:C_0402_1005Metric_Pad0.74x0.62mm_HandSolder, B.Cu at (140.6, 105.7)
- added C6: 100n, Capacitor_SMD:C_0603_1608Metric_Pad1.08x0.95mm_HandSolder, B.Cu at (167.5, 106.0)
- added C7: 100n, Capacitor_SMD:C_0603_1608Metric_Pad1.08x0.95mm_HandSolder, F.Cu at (162.8, 117.4)
- added C8: 10u 35V, Capacitor_SMD:C_1206_3216Metric_Pad1.33x1.80mm_HandSolder, B.Cu at (140.5, 120.8)
- added C9: 100n, Capacitor_SMD:C_0603_1608Metric_Pad1.08x0.95mm_HandSolder, B.Cu at (155.8, 111.5)
- added D1: LED orange, Connector_PinHeader_2.54mm:PinHeader_1x02_P2.54mm_Vertical, F.Cu at (128.2, 76.5)
- added D10: ESD5Zxx, Diode_SMD:D_SOD-523, B.Cu at (174.9, 102.5)
- added D11: TVS (P6SMB16CA), Diode_SMD:D_SMB_Handsoldering, F.Cu at (145.2, 125.5)
- added D12: B260S1F-7, Diode_SMD:D_SOD-123, F.Cu at (141.8, 128.0)
- added D13: ESD5Zxx, Diode_SMD:D_SOD-523, F.Cu at (130.5, 125.8)
- added D14: ESD5Zxx, Diode_SMD:D_SOD-523, F.Cu at (169.5, 125.8)
- added D15: TVS (SMBJ26A), Diode_SMD:D_SMB_Handsoldering, B.Cu at (135.5, 132.8)
- added D16: ESD5Zxx, Diode_SMD:D_SOD-523, F.Cu at (151.7, 105.5)
- added D17: ESD5Zxx, Diode_SMD:D_SOD-523, F.Cu at (154.4, 102.5)
- added D18: ESD5Zxx, Diode_SMD:D_SOD-523, F.Cu at (154.4, 105.5)
- added D19: ESD5Zxx, Diode_SMD:D_SOD-523, F.Cu at (154.4, 104.0)
- added D2: LED orange, Connector_PinHeader_2.54mm:PinHeader_1x02_P2.54mm_Vertical, F.Cu at (169.2, 76.5)
- added D20: ESD5Zxx, Diode_SMD:D_SOD-523, F.Cu at (154.4, 99.8)
- added D21: ESD5Zxx, Diode_SMD:D_SOD-523, F.Cu at (180.0, 136.5)
- added D22: ESD5Zxx, Diode_SMD:D_SOD-523, F.Cu at (180.5, 122.5)
- added D23: ESD5Zxx, Diode_SMD:D_SOD-523, F.Cu at (180.5, 125.0)
- added D24: ESD5Zxx, Diode_SMD:D_SOD-523, F.Cu at (180.5, 127.5)
- added D3: OSRPMC3132A, Connector_PinHeader_2.54mm:PinHeader_1x03_P2.54mm_Vertical, F.Cu at (147.5, 76.5)
- added D4: ES1D, Diode_SMD:D_SMA_Handsoldering, B.Cu at (129.4, 109.2)
- added D5: TVS TPSMB62A, Diode_SMD:D_SMF, B.Cu at (132.4, 102.5)
- added D6: ESD5Zxx, Diode_SMD:D_SOD-523, B.Cu at (174.9, 108.5)
- added D7: ESD5Zxx, Diode_SMD:D_SOD-523, B.Cu at (174.9, 107.0)
- added D8: ESD5Zxx, Diode_SMD:D_SOD-523, B.Cu at (174.9, 105.5)
- added D9: ESD5Zxx, Diode_SMD:D_SOD-523, B.Cu at (174.9, 104.0)
- added F1: Schurter 3403.0155.24, Fuse:Fuse_Schurter_UMT250, B.Cu at (125.1, 104.2)
- added F2: C2Q 300, Fuse:Fuse_0603_1608Metric_Pad1.05x0.95mm_HandSolder, F.Cu at (142.8, 131.2)
- added F3: Mini-Kfz 3A, extraFootprints:KEYSTONE-FUSE-3557-2, B.Cu at (128.0, 126.8)
- added H1: MountingHole, MountingHole:MountingHole_3.2mm_M3_ISO14580, F.Cu at (120.5, 117.5)
- added H2: MountingHole, MountingHole:MountingHole_3.2mm_M3_ISO14580, F.Cu at (120.5, 142.5)
- added H3: MountingHole, MountingHole:MountingHole_3.2mm_M3_ISO14580, F.Cu at (179.5, 117.5)
- added H4: MountingHole, MountingHole:MountingHole_3.2mm_M3_ISO14580, F.Cu at (179.5, 142.5)
- added J1: Photoresistor, Connector_Molex:Molex_PicoBlade_53047-0210_1x02_P1.25mm_Vertical, B.Cu at (178.2, 131.8)
- added J2: Vibration, Connector_Molex:Molex_PicoBlade_53047-0210_1x02_P1.25mm_Vertical, B.Cu at (178.3, 137.1)
- added J3: ESP, Connector_Molex:Molex_PicoBlade_53047-0410_1x04_P1.25mm_Vertical, B.Cu at (178.2, 126.4)
- added J4: ButtonPCB, Connector_Molex:Molex_PicoBlade_53047-0610_1x06_P1.25mm_Vertical, B.Cu at (178.2, 109.2)
- added J5: SWD, Connector_PinHeader_1.27mm:PinHeader_2x05_P1.27mm_Vertical_SMD, B.Cu at (152.4, 102.8)
- added J6: XT30, Connector_AMASS:AMASS_XT30U-M_1x02_P5.0mm_Vertical, B.Cu at (127.5, 134.5)
- added J7: LED strip, Connector_Molex:Molex_PicoBlade_53047-0410_1x04_P1.25mm_Vertical, B.Cu at (136.9, 143.2)
- added JP1: SolderJumper, Jumper:SolderJumper-2_P1.3mm_Open_TrianglePad1.0x1.5mm, B.Cu at (177.6, 83.1)
- added L1: 390u (SRR7045-391M), Inductor_SMD:L_7.3x7.3_H4.5, B.Cu at (133.6, 117.7)
- added L2: 10u, Inductor_SMD:L_1210_3225Metric, F.Cu at (156.0, 128.2)
- added L3: 10u, Inductor_SMD:L_1210_3225Metric, F.Cu at (166.0, 128.3)
- added Q1: BC846C, Package_TO_SOT_SMD:SOT-23_Handsoldering, F.Cu at (144.7, 118.7)
- added Q10: BC846, Package_TO_SOT_SMD:SOT-23_Handsoldering, B.Cu at (156.0, 92.8)
- added Q11: BC856, Package_TO_SOT_SMD:SOT-23_Handsoldering, B.Cu at (156.0, 84.0)
- added Q12: BC846, Package_TO_SOT_SMD:SOT-23_Handsoldering, B.Cu at (164.0, 92.8)
- added Q13: BC856, Package_TO_SOT_SMD:SOT-23_Handsoldering, B.Cu at (164.0, 84.0)
- added Q14: BC846, Package_TO_SOT_SMD:SOT-23_Handsoldering, B.Cu at (170.0, 92.8)
- added Q15: BC856, Package_TO_SOT_SMD:SOT-23_Handsoldering, B.Cu at (170.0, 84.0)
- added Q17: IRLML0030, Package_TO_SOT_SMD:SOT-23_Handsoldering, F.Cu at (135.6, 138.8)
- added Q18: IRLML0030, Package_TO_SOT_SMD:SOT-23_Handsoldering, F.Cu at (131.8, 138.8)
- added Q19: CSD17306Q5A, Package_TO_SOT_SMD:TDSON-8-1, B.Cu at (148.4, 124.0)
- added Q2: FDN306P, Package_TO_SOT_SMD:SOT-23_Handsoldering, F.Cu at (149.4, 117.8)
- added Q3: FDS2734, Package_SO:SOIC-8_3.9x4.9mm_P1.27mm, B.Cu at (126.4, 117.5)
- added Q4: BC846, Package_TO_SOT_SMD:SOT-23_Handsoldering, B.Cu at (132.0, 92.8)
- added Q5: BC856, Package_TO_SOT_SMD:SOT-23_Handsoldering, B.Cu at (132.0, 84.0)
- added Q6: BC846, Package_TO_SOT_SMD:SOT-23_Handsoldering, B.Cu at (140.0, 92.8)
- added Q7: BC856, Package_TO_SOT_SMD:SOT-23_Handsoldering, B.Cu at (140.0, 84.0)
- added Q8: BC846, Package_TO_SOT_SMD:SOT-23_Handsoldering, B.Cu at (148.0, 92.8)
- added Q9: BC856, Package_TO_SOT_SMD:SOT-23_Handsoldering, B.Cu at (148.0, 84.0)
- added R1: R, Resistor_SMD:R_0603_1608Metric_Pad0.98x0.95mm_HandSolder, B.Cu at (133.5, 76.7)
- added R10: 22, Resistor_SMD:R_0603_1608Metric_Pad0.98x0.95mm_HandSolder, B.Cu at (134.3, 111.4)
- added R11: 22k, Resistor_SMD:R_0603_1608Metric_Pad0.98x0.95mm_HandSolder, F.Cu at (149.4, 113.3)
- added R12: 11k, Resistor_SMD:R_0603_1608Metric_Pad0.98x0.95mm_HandSolder, F.Cu at (151.0, 113.3)
- added R13: 680m, Resistor_SMD:R_0603_1608Metric_Pad0.98x0.95mm_HandSolder, B.Cu at (128.1, 122.4)
- added R14: 270k, Resistor_SMD:R_0603_1608Metric_Pad0.98x0.95mm_HandSolder, B.Cu at (140.1, 114.2)
- added R15: 13k, Resistor_SMD:R_0603_1608Metric_Pad0.98x0.95mm_HandSolder, B.Cu at (143.5, 114.2)
- added R16: 330k, Resistor_SMD:R_0603_1608Metric_Pad0.98x0.95mm_HandSolder, F.Cu at (169.5, 115.2)
- added R17: 47k, Resistor_SMD:R_0603_1608Metric_Pad0.98x0.95mm_HandSolder, F.Cu at (173.0, 115.2)
- added R18: 100k, Resistor_SMD:R_0603_1608Metric_Pad0.98x0.95mm_HandSolder, F.Cu at (166.2, 118.8)
- added R19: 5k6, Resistor_SMD:R_0603_1608Metric_Pad0.98x0.95mm_HandSolder, B.Cu at (176.1, 94.0)
- added R2: 10k, Resistor_SMD:R_0603_1608Metric_Pad0.98x0.95mm_HandSolder, B.Cu at (136.8, 103.7)
- added R20: 100k, Resistor_SMD:R_0603_1608Metric_Pad0.98x0.95mm_HandSolder, B.Cu at (177.3, 95.6)
- added R21: 2k2, Resistor_SMD:R_0603_1608Metric_Pad0.98x0.95mm_HandSolder, F.Cu at (158.6, 137.6)
- added R22: 2k2, Resistor_SMD:R_0603_1608Metric_Pad0.98x0.95mm_HandSolder, F.Cu at (161.2, 137.6)
- added R23: 10k, Resistor_SMD:R_0603_1608Metric_Pad0.98x0.95mm_HandSolder, B.Cu at (133.0, 97.3)
- added R24: 220k, Resistor_SMD:R_0603_1608Metric_Pad0.98x0.95mm_HandSolder, B.Cu at (132.1, 87.6)
- added R25: 100k, Resistor_SMD:R_0603_1608Metric_Pad0.98x0.95mm_HandSolder, B.Cu at (132.1, 89.2)
- added R26: 10k, Resistor_SMD:R_0603_1608Metric_Pad0.98x0.95mm_HandSolder, B.Cu at (141.0, 97.3)
- added R27: 220k, Resistor_SMD:R_0603_1608Metric_Pad0.98x0.95mm_HandSolder, B.Cu at (140.1, 87.6)
- added R28: 100k, Resistor_SMD:R_0603_1608Metric_Pad0.98x0.95mm_HandSolder, B.Cu at (140.1, 89.2)
- added R29: 10k, Resistor_SMD:R_0603_1608Metric_Pad0.98x0.95mm_HandSolder, B.Cu at (149.0, 97.3)
- added R3: R, Resistor_SMD:R_0603_1608Metric_Pad0.98x0.95mm_HandSolder, B.Cu at (174.5, 76.5)
- added R30: 220k, Resistor_SMD:R_0603_1608Metric_Pad0.98x0.95mm_HandSolder, B.Cu at (148.1, 87.6)
- added R31: 100k, Resistor_SMD:R_0603_1608Metric_Pad0.98x0.95mm_HandSolder, B.Cu at (148.1, 89.2)
- added R32: 10k, Resistor_SMD:R_0603_1608Metric_Pad0.98x0.95mm_HandSolder, B.Cu at (157.0, 97.3)
- added R33: 220k, Resistor_SMD:R_0603_1608Metric_Pad0.98x0.95mm_HandSolder, B.Cu at (156.1, 87.6)
- added R34: 100k, Resistor_SMD:R_0603_1608Metric_Pad0.98x0.95mm_HandSolder, B.Cu at (156.1, 89.2)
- added R35: 10k, Resistor_SMD:R_0603_1608Metric_Pad0.98x0.95mm_HandSolder, B.Cu at (165.0, 97.3)
- added R36: 220k, Resistor_SMD:R_0603_1608Metric_Pad0.98x0.95mm_HandSolder, B.Cu at (164.1, 87.6)
- added R37: 100k, Resistor_SMD:R_0603_1608Metric_Pad0.98x0.95mm_HandSolder, B.Cu at (164.1, 89.2)
- added R38: 10k, Resistor_SMD:R_0603_1608Metric_Pad0.98x0.95mm_HandSolder, B.Cu at (171.0, 97.3)
- added R39: 220k, Resistor_SMD:R_0603_1608Metric_Pad0.98x0.95mm_HandSolder, B.Cu at (170.1, 87.6)
- added R4: 24k3, Resistor_SMD:R_0603_1608Metric_Pad0.98x0.95mm_HandSolder, B.Cu at (144.1, 110.2)
- added R40: 100k, Resistor_SMD:R_0603_1608Metric_Pad0.98x0.95mm_HandSolder, B.Cu at (170.1, 89.2)
- added R41: 100R, Resistor_SMD:R_0603_1608Metric_Pad0.98x0.95mm_HandSolder, F.Cu at (136.6, 132.7)
- added R42: 1M, Resistor_SMD:R_0603_1608Metric_Pad0.98x0.95mm_HandSolder, F.Cu at (135.7, 135.2)
- added R43: 100R, Resistor_SMD:R_0603_1608Metric_Pad0.98x0.95mm_HandSolder, F.Cu at (132.8, 132.8)
- added R44: 1M, Resistor_SMD:R_0603_1608Metric_Pad0.98x0.95mm_HandSolder, F.Cu at (131.9, 135.3)
- added R45: 4k7 1%, Resistor_SMD:R_0603_1608Metric_Pad0.98x0.95mm_HandSolder, F.Cu at (150.5, 133.2)
- added R46: 1k5 1%, Resistor_SMD:R_0603_1608Metric_Pad0.98x0.95mm_HandSolder, F.Cu at (150.5, 135.0)
- added R47: 4k7 1%, Resistor_SMD:R_0603_1608Metric_Pad0.98x0.95mm_HandSolder, F.Cu at (160.5, 133.3)
- added R48: 1k5 1%, Resistor_SMD:R_0603_1608Metric_Pad0.98x0.95mm_HandSolder, F.Cu at (160.5, 135.0)
- added R5: 56k, Resistor_SMD:R_0603_1608Metric_Pad0.98x0.95mm_HandSolder, B.Cu at (142.3, 105.7)
- added R6: 68R, Resistor_SMD:R_0603_1608Metric_Pad0.98x0.95mm_HandSolder, B.Cu at (144.8, 76.8)
- added R7: 4R7, Resistor_SMD:R_0603_1608Metric_Pad0.98x0.95mm_HandSolder, B.Cu at (155.2, 76.8)
- added R8: 100k, Resistor_SMD:R_0603_1608Metric_Pad0.98x0.95mm_HandSolder, F.Cu at (141.0, 118.7)
- added R9: 100k, Resistor_SMD:R_0603_1608Metric_Pad0.98x0.95mm_HandSolder, F.Cu at (149.3, 121.5)
- added SW1: SW_Left, Button_Switch_SMD:SW_SPST_PTS810, F.Cu at (126.8, 125.8)
- added SW2: SW_Right, Button_Switch_SMD:SW_SPST_PTS810, F.Cu at (173.2, 125.8)
- added SW3: Reset, Button_Switch_SMD:SW_SPST_PTS810, F.Cu at (171.7, 142.2)
- added U1: LT3757AEMSE, Package_SO:MSOP-10-1EP_3x3mm_P0.5mm_EP1.68x1.88mm, B.Cu at (138.2, 108.7)
- added U2: STM32L433CCTx, Package_QFP:LQFP-48_7x7mm_P0.5mm, F.Cu at (162.0, 110.0)
- added U3: HV5812, Package_SO:SOIC-28W_7.5x17.9mm_P1.27mm, F.Cu at (150.0, 90.7)
- added U4: MIC4801, Package_SO:PowerIntegrations_SO-8, B.Cu at (177.7, 89.0)
- added U5: DS3231-module, extraFootprints:DS3231-module, B.Cu at (159.9, 140.2)
- added U6: LM74700, Package_TO_SOT_SMD:SOT-23-6, B.Cu at (143.1, 126.9)
- added U7: TPS62175DQC, Package_SON:WSON-10-1EP_2x3mm_P0.5mm_EP0.84x2.4mm_ThermalVias, F.Cu at (152.6, 130.2)
- added U8: TPS62175DQC, Package_SON:WSON-10-1EP_2x3mm_P0.5mm_EP0.84x2.4mm_ThermalVias, F.Cu at (162.6, 130.3)
- added V1: SVM-06SS33, extraFootprints:SVM-06SS33, F.Cu at (150.0, 100.0)
Routing:
- net +3V3: track 0.00 -> 224.0 mm, vias 0 -> 14
- net GND: track 0.00 -> 219.2 mm, vias 0 -> 258
- net Vdrive: track 0.00 -> 101.7 mm, vias 0 -> 1
- net /Alarm1_LED: track 0.00 -> 98.5 mm, vias 0 -> 1
- net +24V: track 0.00 -> 77.9 mm, vias 0 -> 3
- net /Status_LED_Red: track 0.00 -> 73.7 mm, vias 0 -> 1
- net VDC: track 0.00 -> 73.6 mm, vias 0 -> 7
- net /Alarm2_LED: track 0.00 -> 63.5 mm, vias 0 -> 1
- net /Status_LED_Green: track 0.00 -> 60.8 mm, vias 0 -> 1
- net /~{RST}: track 0.00 -> 57.0 mm, vias 0 -> 6
- net /Button.Left: track 0.00 -> 43.5 mm, vias 0 -> 2
- net /enableWarmWhite: track 0.00 -> 40.8 mm, vias 0 -> 2
- net /enableColdWhite: track 0.00 -> 40.6 mm, vias 0 -> 2
- net Net-(D4-A): track 0.00 -> 40.4 mm
- net /Vibration: track 0.00 -> 36.3 mm, vias 0 -> 2
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- added copper zone on B.Cu, net GND
- added copper zone on F.Cu, net GND
Other:
- board outline added: 65 x 71.5 mm
- board text added: "alarm-clock v3 2024-06 by MG-5"

Commit message: Polish
Parts:
- added TP1: 35V, TestPoint:TestPoint_THTPad_D1.5mm_Drill0.7mm, F.Cu at (119.8, 108.5)
- added TP2: GND, TestPoint:TestPoint_THTPad_D1.5mm_Drill0.7mm, F.Cu at (126.5, 141.5)
Routing:
- net Vdrive: track 101.7 -> 107.7 mm
- net Net-(D4-K): track 27.6 -> 32.6 mm
- net +9V: track 22.6 -> 19.7 mm
- net VDC: track 73.6 -> 71.1 mm
- net GND: track 219.2 -> 216.7 mm, vias 258 -> 257
- net /Button.Left: track 43.5 -> 41.7 mm
- net /I2C1_SDA: track 32.9 -> 31.1 mm
- net +24V: track 77.9 -> 79.5 mm
- net Net-(Q3-S-Pad1): track 21.6 -> 19.9 mm
- net /F: track 7.39 -> 5.92 mm
- net /I2C1_SCL: track 32.4 -> 31.1 mm
- net /enable35V: track 32.6 -> 31.5 mm
- net /G1: track 12.4 -> 11.3 mm
- net /~{RST}: track 57.0 -> 55.9 mm
- net +3V3: track 224.0 -> 222.9 mm
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Other:
- board text added: "35V"
- board text added: "GND"

Commit message: Gerber settings
Other:
- board text added: "JLCJLCJLCJLC"
Changed lines of the file:
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@@
 			(plot_on_all_layers_selection 0x0000000_00000000)
 			(disableapertmacros no)
-			(usegerberextensions no)
+			(usegerberextensions yes)
 			(usegerberattributes yes)
 			(usegerberadvancedattributes yes)
-			(creategerberjobfile yes)
+			(creategerberjobfile no)
 			(dashed_line_dash_ratio 12.000000)
 			(dashed_line_gap_ratio 3.000000)
@@
 			(plotinvisibletext no)
 			(sketchpadsonfab no)
-			(subtractmaskfromsilk no)
+			(subtractmaskfromsilk yes)
 			(outputformat 1)
 			(mirror no)
-			(drillshape 1)
+			(drillshape 0)
 			(scaleselection 1)
-			(outputdirectory "")
+			(outputdirectory "gerber")
 		)
 	)
@@
 		(layer "B.SilkS")
 		(effects
+			(font
+				(size 0.8 0.8)
+				(thickness 0.1)
+			)
+			(justify left bottom mirror)
+		)
+	)
+	(gr_text "JLCJLCJLCJLC"
+		(at 163.75 124.25 -0)
+		(layer "B.SilkS")
+		(effects
